File: Kicad/JLCTestProjekt1/JLCTestProjekt1.kicad_sch (KiCad schematic)
At the start: 5 parts, among them J1 Analog, J2 Digital, SW1 SW_Push

Commit message: Footprint korrigiert und MPN als Eigenschaft
Parts:
- D1: JLCPCB C49018 -> (none); MPN (none) -> C49018
- R1: footprint Capacitor_SMD:C_0805_2012Metric -> Resistor_SMD:R_0805_2012Metric; JLCPCB C4256393 -> (none); MPN (none) -> C4256393
- SW1: JLCPCB C2921128 -> (none); MPN (none) -> C2921128
Changed lines of the file:
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@@
 			)
 		)
-		(property "Footprint" "Capacitor_SMD:C_0805_2012Metric"
+		(property "Footprint" "Resistor_SMD:R_0805_2012Metric"
 			(at 150.622 62.23 90)
 			(effects
@@
 			)
 		)
-		(property "JLCPCB" "C4256393"
+		(property "MPN" "C4256393"
 			(at 150.114 62.23 90)
 			(effects
@@
 			)
 		)
-		(property "JLCPCB" "C2921128"
+		(property "MPN" "C2921128"
 			(at 129.54 52.832 0)
 			(effects
@@
 			)
 		)
-		(property "JLCPCB" "C49018"
+		(property "MPN" "C49018"
 			(at 146.05 53.594 0)
 			(effects
